File: CAN_IMU.kicad_pcb (KiCad board)
At the start: 2 copper layers, 77 x 61.5 mm, 36 parts, among them J1 USB_C_Receptacle_USB2.0_16P, J2 TAG SWD, J3 Conn_01x05, SW1 RST, SW2 SW_DIP_x02, U1 STM32G431CBTx, U2 USBLC6-2SC6, U3 SN74LVC1G126DBV, U4 TCAN3414, U5 TPS62172DSG

Commit message: Basically finished layout
Parts:
- added R8: 47k, Resistor_SMD:R_0603_1608Metric, F.Cu at (44.8, 64.0)
- C7: value 2.2uF -> 10uF
- L1: value 10uH -> 2.2uH; footprint Inductor_SMD:L_Bourns-SRN6028 -> RJMP_Inductors:IND_LQH5BPN2R2NT0L
- moved R5 67.1 mm to (72.6, 86.5), turned to -90 degrees
- moved C10 66.6 mm to (75.8, 69.5), turned to 90 degrees
- moved R7 66.0 mm to (74.1, 86.5), turned to -90 degrees
- moved C2 65.5 mm to (71.0, 68.2), turned to -90 degrees
- moved R6 64.5 mm to (71.1, 86.5), turned to -90 degrees
- moved C4 63.9 mm to (68.2, 77.5), turned to 180 degrees
- moved R2 61.6 mm to (65.0, 89.3), turned to 90 degrees
- moved C5 60.3 mm to (65.3, 77.5), turned to 180 degrees
- moved R4 60.3 mm to (67.0, 87.0), turned to -90 degrees
- moved C1 59.2 mm to (56.2, 85.0), turned to -90 degrees
- moved R1 56.5 mm to (55.5, 92.0), turned to 90 degrees
- moved C3 55.4 mm to (61.7, 65.0)
- moved U1 54.3 mm to (64.8, 71.2)
- moved D3 52.7 mm to (73.8, 48.9)
- moved C6 51.9 mm to (58.6, 68.1), turned to 90 degrees
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Connections:
- net Net-(U5-SW) renamed /SW
- D2 pad 1: /CAN_L -> /CAN_H
- D2 pad 2: /CAN_H -> /CAN_L
- J2 pad 1: VDD -> VCC
- U1 pad 10: /IMU_GPIO3 -> unconnected-(U1-PA2-Pad10)
- U1 pad 11: /IMU_GPIO4 -> unconnected-(U1-PA3-Pad11)
- U1 pad 12: unconnected-(U1-PA4-Pad12) -> /MODE_SW
- U1 pad 13: /CAN_SHDN -> unconnected-(U1-PA5-Pad13)
- U1 pad 14: /CAN_STBY -> unconnected-(U1-PA6-Pad14)
- U1 pad 16: /CAN_RX_EN -> unconnected-(U1-PB0-Pad16)
- U1 pad 25: unconnected-(U1-PB11-Pad25) -> /IMU_GPIO3
- U1 pad 26: unconnected-(U1-PB12-Pad26) -> /IMU_GPIO4
- U1 pad 27: unconnected-(U1-PB13-Pad27) -> /IMU_GPIO2
- U1 pad 28: unconnected-(U1-PB14-Pad28) -> /IMU_GPIO1
- U1 pad 41: unconnected-(U1-PB4-Pad41) -> /CAN_SHDN
- U1 pad 43: unconnected-(U1-PB6-Pad43) -> /CAN_STBY
- U1 pad 44: unconnected-(U1-PB7-Pad44) -> /CAN_RX_EN
- U1 pad 8: /IMU_GPIO1 -> unconnected-(U1-PA0-Pad8)
- U1 pad 9: /IMU_GPIO2 -> unconnected-(U1-PA1-Pad9)
Routing:
- net VBUS: track 0.00 -> 78.8 mm
- net GND: track 0.00 -> 56.2 mm, vias 0 -> 31
- net /CAN_RX-BOOT0: track 0.00 -> 31.1 mm
- net VCC: track 0.00 -> 29.8 mm, vias 0 -> 11
- net /SWO: track 0.00 -> 29.8 mm, vias 0 -> 2
- net /SWCLK: track 0.00 -> 27.5 mm, vias 0 -> 2
- net /NRST: track 0.00 -> 25.8 mm, vias 0 -> 2
- net /SWDIO: track 0.00 -> 25.7 mm, vias 0 -> 2
- net /IMU_GPIO3: track 0.00 -> 24.4 mm
- net /CAN_STBY: track 0.00 -> 22.9 mm
- net /CAN_TX: track 0.00 -> 22.8 mm, vias 0 -> 2
- net /USB_DP: track 0.00 -> 22.7 mm
- net /CAN_RX_EN: track 0.00 -> 22.0 mm
- net /USB_DM: track 0.00 -> 21.5 mm
- net /CAN_L: track 0.00 -> 20.9 mm
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- added copper zone on F.Cu, net /SW
- added copper zone on In2.Cu, net /VUSB
- added copper zone on B.Cu, net GND
- added copper zone on F.Cu, net GND
- added copper zone on In1.Cu, net GND
- added copper zone on F.Cu, net VBUS
- added copper zone on F.Cu, net VCC
- added copper zone on In2.Cu, net VCC
Other:
- copper layers 2 -> 4
- board text added: "DFU"
- board text added: "G"
- board text added: "H"
- board text added: "L"
- board text added: "NMEA"
- board text added: "RESET"
- board text added: "S"
- board text added: "V"
