File: onboard_imu.kicad_sch (KiCad schematic)
At the start: 15 parts, among them U10 SN74AUP1T34DCK, U7 ICM-20948, U8 MCP1700x-180xxTT, U9 SN74AUP1T34DCK

Commit message: Fix some missing part numbers and update BOM
No artwork changes.
Parts:
- U10, U9: LCSC Part Number (none) -> C131985
- U7: Digikey Part Number (none) -> 1428-1123-1-ND; LCSC Part Number (none) -> C726001; Mfg Part Number (none) -> ICM-20948
- U8: Digikey Part Number (none) -> MCP1700T1802ETTCT-ND; LCSC Part Number (none) -> C150796; Mfg Part Number (none) -> MCP1700T-1802E/TT
Changed lines of the file:
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@@
+			)
+		)
+		(property "Mfg Part Number" "MCP1700T-1802E/TT"
+			(at 73.66 44.45 0)
+			(effects
+				(font
+					(size 1.27 1.27)
+				)
+				(hide yes)
+			)
+		)
+		(property "Digikey Part Number" "MCP1700T1802ETTCT-ND"
+			(at 73.66 44.45 0)
+			(effects
+				(font
+					(size 1.27 1.27)
+				)
+				(hide yes)
+			)
+		)
+		(property "LCSC Part Number" "C150796"
+			(at 73.66 44.45 0)
+			(effects
+				(font
+					(size 1.27 1.27)
+				)
+				(hide yes)
 			)
 		)
@@
 			)
 		)
+		(property "LCSC Part Number" "C131985"
+			(at 167.64 53.34 0)
+			(effects
+				(font
+					(size 1.27 1.27)
+				)
+				(hide yes)
+			)
+		)
 		(pin "3"
 		)
@@
 			)
 		)
+		(property "LCSC Part Number" "C131985"
+			(at 167.64 120.65 0)
+			(effects
+				(font
+					(size 1.27 1.27)
+				)
+				(hide yes)
+			)
+		)
 		(pin "3"
 		)
@@
 			(at 125.73 87.63 0)
 			(effects
+				(font
+					(size 1.27 1.27)
+				)
+				(hide yes)
+			)
+		)
+		(property "Mfg Part Number" "ICM-20948"
+			(at 125.73 87.63 0)
+			(effects
+				(font
+					(size 1.27 1.27)
+				)
+				(hide yes)
+			)
+		)
+		(property "Digikey Part Number" "1428-1123-1-ND"
+			(at 125.73 87.63 0)
+			(effects
+				(font
+					(size 1.27 1.27)
+				)
+				(hide yes)
+			)
+		)
+		(property "LCSC Part Number" "C726001"
+			(at 125.73 87.63 0)
+			(effects
